File: PF-2026/PF-2026-1.kicad_sch (KiCad schematic)
At the start: 37 parts, among them U1 ATMEGA328P-AU, Y1 ABM8-16.000MHZ

Commit message: Finalise PCB design
Parts:
- removed D1: PESD5V0U1BB, bc-protection:PESDX_R, symbol bc-protection:D-PESD5V0U1BB
- removed TP13: ~, bh-testpoint:TP-1.0-MM, symbol bh-testpoint:TP-1.0-MM
Connections:
- net +5V: now also D2.2; no longer D2.A
- net at C1.1, C2.1, R1.2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: now also D2.1; no longer D2.C
