File: PF-2026/PF-2026-3.kicad_sch (KiCad schematic)
At the start: 57 parts

Commit message: Finalise PCB design
Parts:
- removed C44, C45, C46, C47, C48, C49, C50, C51, C52, C53, C54, C55, C56, C57, C58, C59, C60: 100nF, bh-capacitor:CAPACITOR-0402_R, symbol bh-capacitor:C-0402-100NF
- removed LED40, LED41, LED42, LED43, LED44, LED45, LED46, LED47, LED48, LED49, LED50, LED51, LED52, LED53, LED54, LED55, LED56: WS2812B-2020, bc-led:WS2812B-2020_R, symbol bc-led:LED-WS2812B-2020
- removed R5: 330R, bh-resistor:RESISTOR-0402_R, symbol bh-resistor:R-0402-330R
Connections:
- net LED: now also LED29.3 (DI)
Other:
- moved on the sheet: C33, C34, C35, C36, C37, C38, C39, C40, C41, C42, C43, LED29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
