File: PF-2026/PF-2026.kicad_pcb (KiCad board)
At the start: 2 copper layers, 151 parts, among them U1 ATMEGA328P-AU, Y1 ABM8-16.000MHZ

Commit message: Finalise PCB design
Parts:
- removed C44, C45, C46, C47, C48, C49, C50, C51, C52, C53, C54, C55, C56, C57, C58, C59, C60: 100nF, bh-capacitor:CAPACITOR-0402_R
- removed D1: PESD5V0U1BB, bc-protection:PESDX_R
- removed LED40, LED41, LED42, LED43, LED44, LED45, LED46, LED47, LED48, LED49, LED50, LED51, LED52, LED53, LED54, LED55, LED56: WS2812B-2020, bc-led:WS2812B-2020_R
- removed R5: 330R, bh-resistor:RESISTOR-0402_R
- removed TP13: ~, bh-testpoint:TP-1.0-MM
- added kibuzzard-69414ECA: G***, kibuzzard-69414ECA, F.Cu at (35.8, 24.0)
- added kibuzzard-69414ECA: G***, kibuzzard-69414ECA, F.Cu at (23.4, 24.0)
- added kibuzzard-69414EE3: G***, kibuzzard-69414EE3, F.Cu at (33.3, 24.0)
- added kibuzzard-69414EEA: G***, kibuzzard-69414EEA, F.Cu at (30.7, 24.0)
- added kibuzzard-69414EF3: G***, kibuzzard-69414EF3, F.Cu at (10.7, 24.0)
- added kibuzzard-69414EF3: G***, kibuzzard-69414EF3, F.Cu at (28.2, 24.0)
- added kibuzzard-69414F1E: G***, kibuzzard-69414F1E, F.Cu at (20.8, 24.0)
- added kibuzzard-69414F25: G***, kibuzzard-69414F25, F.Cu at (18.3, 24.0)
- added kibuzzard-69414F2A: G***, kibuzzard-69414F2A, F.Cu at (15.7, 24.0)
- added kibuzzard-69414F2F: G***, kibuzzard-69414F2F, F.Cu at (13.2, 24.0)
- TP1, TP10, TP11, TP12, TP14, TP15, TP16, TP17, TP18, TP19, TP2, TP20, TP21, TP22, TP3, TP4, TP5, TP6, TP7, TP8, TP9: moved to B.Cu
- moved LED36 69.0 mm to (36.5, 6.50), turned to 145 degrees
- moved R4 62.7 mm to (-7.45, 13.2), turned to 180 degrees
- moved LED37 61.1 mm to (37.4, 2.40), turned to 180 degrees
- moved C41 59.2 mm to (37.4, 0.40), turned to 180 degrees
- moved JP3 58.5 mm to (32.0, 28.0), turned to 90 degrees
- moved LED29 57.1 mm to (35.8, -10.0), turned to -95 degrees
- moved C38 55.7 mm to (29.8, 8.10), turned to 60 degrees
- moved C39 54.3 mm to (34.7, 8.00), turned to 120 degrees
- moved C37 53.9 mm to (27.0, 4.40)
- moved C42 53.3 mm to (34.5, -3.00), turned to -120 degrees
- moved LED38 52.6 mm to (36.2, -1.70), turned to -140 degrees
- moved C36 51.4 mm to (26.9, -0.20)
- moved C43 50.9 mm to (29.7, -2.80), turned to -60 degrees
- moved LED30 50.7 mm to (31.4, -9.60), turned to -60 degrees
- moved TP11 50.0 mm to (33.3, 25.0), turned to 180 degrees
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Connections:
- D2 pad 1: (no net) -> Net-(U1-AREF)
- D2 pad 2: (no net) -> +5V
- LED29 pad 3: Net-(LED29-DI) -> LED
- LED39 pad 1: Net-(LED39-DO) -> unconnected-(LED39-DO-Pad1)
- R4 pad 1: IO -> IO3
- U1 pad 1: /MCU/IO3 -> IO3
Routing:
- net +5V: track 0.00 -> 123.4 mm, vias 0 -> 41
- net /MCU/RESET: track 0.00 -> 61.2 mm, vias 0 -> 1
- net /MCU/RXD: track 0.00 -> 52.5 mm, vias 0 -> 1
- net /MCU/TXD: track 0.00 -> 46.6 mm, vias 0 -> 1
- net LED: track 0.00 -> 36.8 mm, vias 0 -> 2
- net Net-(U1-AREF): track 0.00 -> 30.9 mm, vias 0 -> 1
- net Net-(LED1-DI): track 0.00 -> 30.8 mm, vias 0 -> 2
- net /MCU/MISO: track 0.00 -> 24.9 mm, vias 0 -> 1
- net Net-(LED18-DO): track 0.00 -> 23.9 mm, vias 0 -> 2
- net Net-(LED10-DO): track 0.00 -> 23.7 mm, vias 0 -> 2
- net /MCU/MOSI: track 0.00 -> 23.1 mm, vias 0 -> 1
- net /MCU/SCK: track 0.00 -> 17.6 mm, vias 0 -> 1
- net Net-(LED14-DO): track 0.00 -> 11.1 mm, vias 0 -> 2
- net Net-(LED17-DO): track 0.00 -> 9.69 mm, vias 0 -> 2
- net Net-(LED16-DO): track 0.00 -> 9.69 mm, vias 0 -> 2
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- added copper zone on In1.Cu, net +5V
- added copper zone on B.Cu, net GND
- added copper zone on F.Cu, net GND
- added copper zone on In2.Cu, net GND
Other:
- board outline added: 88 x 48 mm
- copper layers 2 -> 4
- board text added: "HAPPY NEW YEAR!"
- board text added: "USB-C"
- board text added: "What exactly did you expect to find here?"
